Commit message: enable choice of different robots

File: kassow_kord_bringup/urdf/kassow_kord.urdf.xacro (robot description, xacro)
@@ -6,12 +6,13 @@
   <xacro:arg name="port" default="28283"/>
   <xacro:arg name="session_id" default="1"/>
+  <xacro:arg name="robot_model" default="kr810"/>
   <xacro:include filename="$(find kassow_kord_bringup)/urdf/common/inertials.xacro" />
   <xacro:include filename="$(find kassow_kord_bringup)/urdf/common/materials.xacro" />
-  <xacro:include filename="$(find kassow_kord_description)/kr810/urdf/kr810_description.urdf.xacro"/>
   <xacro:include filename="$(find kassow_kord_bringup)/urdf/kassow_kord.ros2_control.xacro"/>
   <link name="world"/>
-  <xacro:kr810_description prefix="$(arg prefix)" parent="world">
+  <xacro:include filename="$(find kassow_kord_description)/$(arg robot_model)/urdf/$(arg robot_model)_description.urdf.xacro"/>
+  <xacro:call macro="$(arg robot_model)_description" prefix="$(arg prefix)" parent="world">
     <origin xyz="0 0 0" rpy="0 0 0"/>
-  </xacro:kr810_description>
+  </xacro:call>
   <xacro:kassow_kord_ros2_control
     name="$(arg prefix)"

File: kassow_kord_bringup/urdf/kassow_kord_dual_arm.urdf.xacro (robot description, xacro)
@@ -2,8 +2,10 @@
 <robot xmlns:xacro="http://www.ros.org/wiki/xacro" name="kassow_kord">
   <xacro:arg name="use_mock_hardware" default="true"/>
+  <xacro:arg name="robot_1_model" default="kr810"/>
   <xacro:arg name="robot_1_prefix" default="kassow_right"/>
   <xacro:arg name="robot_1_ip" default="10.23.23.204"/>
   <xacro:arg name="robot_1_port" default="28283"/>
   <xacro:arg name="robot_1_session_id" default="1"/>
+  <xacro:arg name="robot_2_model" default="kr810"/>
   <xacro:arg name="robot_2_prefix" default="kassow_left"/>
   <xacro:arg name="robot_2_ip" default="10.23.23.205"/>
@@ -16,7 +18,8 @@
   <link name="world"/>
   <!-- KASSOW 1 -->
-  <xacro:kr810_description prefix="$(arg robot_1_prefix)" parent="world">
+  <xacro:include filename="$(find kassow_kord_description)/$(arg robot_1_model)/urdf/$(arg robot_1_model)_description.urdf.xacro"/>
+  <xacro:call macro="$(arg robot_1_model)_description" prefix="$(arg robot_1_prefix)" parent="world">
     <origin xyz="0 1.0 0" rpy="0 0 0"/>
-  </xacro:kr810_description>
+  </xacro:call>
   <xacro:kassow_kord_ros2_control
     name="$(arg robot_1_prefix)"
@@ -28,7 +31,8 @@
   />
   <!-- KASSOW 2 -->
-  <xacro:kr810_description prefix="$(arg robot_2_prefix)" parent="world">
+  <xacro:include filename="$(find kassow_kord_description)/$(arg robot_2_model)/urdf/$(arg robot_2_model)_description.urdf.xacro"/>
+  <xacro:call macro="$(arg robot_2_model)_description" prefix="$(arg robot_2_prefix)" parent="world">
     <origin xyz="0 -1.0 0" rpy="0 0 0"/>
-  </xacro:kr810_description>
+  </xacro:call>
   <xacro:kassow_kord_ros2_control
     name="$(arg robot_2_prefix)"

File: kassow_kord_description/kr810/urdf/kr810_description.urdf.xacro (robot description, xacro)
@@ -1,5 +1,5 @@
 <?xml version="1.0" ?>
 <robot name="kr2_robot_a810" model="a810" model-revision="051020-0" mechanical-revision="5" features="TIO" xmlns:xacro="http://www.ros.org/wiki/xacro">
-  <xacro:macro name="kassow_robot" params="prefix parent *origin">
+  <xacro:macro name="kr810_description" params="prefix parent *origin">
   <!-- globals -->
   <xacro:property name="joints_damping" value="0.1" />
