Commit message: bringup tested

File: kassow_kord_bringup/urdf/kassow_kord.ros2_control.xacro (robot description, xacro)
@@ -4,7 +4,11 @@
     <ros2_control name="${name}" type="system">
       <hardware>
-        <plugin>kassow_kord_hardware/KassowKordHardwareInterface</plugin>
+        <plugin>kassow_kord_hardware_interface/KassowKordHardwareInterface</plugin>
+        <param name="ip_address">192.168.1.100</param>
+        <param name="port">7582</param>
+        <param name="session_id">1</param>
+        <param name="waitSync_timeout_ms">500</param>
       </hardware>
-      <joint name="joint1">
+      <joint name="joint_1">
         <command_interface name="position"/>
         <state_interface name="position"/>
@@ -12,5 +16,5 @@
         <state_interface name="effort"/>
       </joint>
-      <joint name="joint2">
+      <joint name="joint_2">
         <command_interface name="position"/>
         <state_interface name="position"/>
@@ -18,5 +22,5 @@
         <state_interface name="effort"/>
       </joint>
-      <joint name="joint3">
+      <joint name="joint_3">
         <command_interface name="position"/>
         <state_interface name="position"/>
@@ -24,5 +28,5 @@
         <state_interface name="effort"/>
       </joint>
-      <joint name="joint4">
+      <joint name="joint_4">
         <command_interface name="position"/>
         <state_interface name="position"/>
@@ -30,5 +34,5 @@
         <state_interface name="effort"/>
       </joint>
-      <joint name="joint5">
+      <joint name="joint_5">
         <command_interface name="position"/>
         <state_interface name="position"/>
@@ -36,5 +40,5 @@
         <state_interface name="effort"/>
       </joint>
-      <joint name="joint6">
+      <joint name="joint_6">
         <command_interface name="position"/>
         <state_interface name="position"/>
@@ -42,5 +46,5 @@
         <state_interface name="effort"/>
       </joint>
-      <joint name="joint7">
+      <joint name="joint_7">
         <command_interface name="position"/>
         <state_interface name="position"/>

File: kassow_kord_bringup/urdf/kassow_kord.urdf.xacro (robot description, xacro)
@@ -5,7 +5,5 @@
   <!-- Minimal 7-DOF serial manipulator URDF (no visuals/collisions) -->
   <!-- Base link -->
-  <link name="base_link">
-    <xacro:default_inertial/>
-  </link>
+  <link name="base_link"/>
   <!-- 7 links + 7 revolute joints -->
   <!-- links spaced along the +X axis by 0.2 m each -->

Commit message: add moveit setup and srdf

File: kassow_kord_bringup/urdf/kassow_kord.ros2_control.xacro (robot description, xacro)
@@ -1,12 +1,17 @@
 <?xml version="1.0"?>
 <robot xmlns:xacro="http://www.ros.org/wiki/xacro">
-  <xacro:macro name="kassow_kord_ros2_control" params="name">
+  <xacro:macro name="kassow_kord_ros2_control" params="name prefix use_mock_hardware:=false">
     <ros2_control name="${name}" type="system">
       <hardware>
-        <plugin>kassow_kord_hardware_interface/KassowKordHardwareInterface</plugin>
-        <param name="ip_address">10.28.28.11</param>
-        <param name="port">7582</param>
-        <param name="session_id">1</param>
-        <param name="waitSync_timeout_ms">500</param>
+        <xacro:if value="$(arg use_mock_hardware)">
+          <plugin>mock_components/GenericSystem</plugin>
+        </xacro:if>
+        <xacro:unless value="$(arg use_mock_hardware)">
+          <plugin>kassow_kord_hardware_interface/KassowKordHardwareInterface</plugin>
+          <param name="ip_address">10.28.28.11</param>
+          <param name="port">7582</param>
+          <param name="session_id">1</param>
+          <param name="waitSync_timeout_ms">500</param>
+        </xacro:unless>
       </hardware>
       <joint name="joint_1">

File: kassow_kord_bringup/urdf/kassow_kord.urdf.xacro (robot description, xacro)
@@ -1,4 +1,6 @@
 <?xml version="1.0"?>
 <robot xmlns:xacro="http://www.ros.org/wiki/xacro" name="kassow_kord">
+  <xacro:arg name="prefix" default=""/>
+  <xacro:arg name="use_mock_hardware" default="false"/>
   <xacro:include filename="$(find kassow_kord_bringup)/urdf/common/inertials.xacro" />
   <xacro:include filename="$(find kassow_kord_description)/kr810/urdf/kr810_description.urdf.xacro"/>
@@ -7,4 +9,7 @@
   <xacro:kr810_description/>
   <!-- Add ros2_control hardware -->
-  <xacro:kassow_kord_ros2_control name="kassow_kord_control"/>
+  <xacro:kassow_kord_ros2_control
+    name="kassow_kord_control"
+    prefix="$(arg prefix)"
+    use_mock_hardware="$(arg use_mock_hardware)"/>
 </robot>

File: kassow_kord_description/kr810/urdf/kr810_description.urdf.xacro (robot description, xacro)
@@ -322,5 +322,5 @@
     <child link="base"/>
   </joint>
-  <joint name="joint_1" type="continuous">
+  <joint name="joint_1" type="revolute">
     <parent link="base"/>
     <child link="link1"/>
@@ -334,5 +334,5 @@
   <xacro:property name="joint1_yoffset"  value="${   0.0 * scale}" />
   <xacro:property name="joint1_zoffset"  value="${ 308.7 * scale - 35 * scale}" />
-  <joint name="joint_2" type="continuous">
+  <joint name="joint_2" type="revolute">
     <parent link="link1"/>
     <child link="linkJ2"/>
@@ -350,5 +350,5 @@
     <origin rpy="0 0 0" xyz="${jointPL2_xoffset} ${jointPL2_yoffset} 0"/>
   </joint>
-  <joint name="joint_3" type="continuous">
+  <joint name="joint_3" type="revolute">
     <parent link="link2"/>
     <child link="link3"/>
@@ -362,5 +362,5 @@
   <xacro:property name="joint3_yoffset"  value="${ 0.0 * scale}" />
   <xacro:property name="joint3_zoffset"  value="${ 142.9 * scale}" />
-  <joint name="joint_4" type="continuous">
+  <joint name="joint_4" type="revolute">
     <parent link="link3"/>
     <child link="linkJ4"/>
@@ -379,5 +379,5 @@
     <origin rpy="0 0 0" xyz="${jointPL4_xoffset} ${jointPL4_yoffset} ${jointPL4_zoffset}"/>
   </joint>
-  <joint name="joint_5" type="continuous">
+  <joint name="joint_5" type="revolute">
     <parent link="link4"/>
     <child link="link5"/>
@@ -389,5 +389,5 @@
   </joint>
   <xacro:property name="joint5_zoffset"  value="${ 103.5 * scale}" />
-  <joint name="joint_6" type="continuous">
+  <joint name="joint_6" type="revolute">
     <parent link="link5"/>
     <child link="linkJ6"/>
@@ -405,5 +405,5 @@
   </joint>
   <xacro:property name="joint6_zoffset"  value="${ 108.0 * scale}" />
-  <joint name="joint_7" type="continuous">
+  <joint name="joint_7" type="revolute">
     <parent link="link6"/>
     <child link="end_effector"/>

Commit message: Update the interface to run on the simulator.

File: kassow_kord_bringup/urdf/kassow_kord.ros2_control.xacro (robot description, xacro)
@@ -1,6 +1,13 @@
 <?xml version="1.0"?>
 <robot xmlns:xacro="http://www.ros.org/wiki/xacro">
-  <xacro:macro name="kassow_kord_ros2_control" params="name prefix use_mock_hardware:=false">
-    <ros2_control name="${name}" type="system">
+  <xacro:macro name="kassow_kord_ros2_control"
+              params="name
+                      prefix
+                      use_mock_hardware:=false
+                      ip_address:=10.28.28.11
+                      port:=7582
+                      session_id:=1"
+                      >
+    <ros2_control name="${name}" type="system" is_async="false" rw_rate="250">
       <hardware>
         <xacro:if value="$(arg use_mock_hardware)">
@@ -9,11 +16,7 @@
         <xacro:unless value="$(arg use_mock_hardware)">
           <plugin>kassow_kord_hardware_interface/KassowKordHardwareInterface</plugin>
-          <param name="ip_address">10.28.28.11</param>
-          <param name="port">7582</param>
-          <param name="session_id">1</param>
-          <param name="waitSync_timeout_ms">500</param>
-          <param name="tracking_time">0.008</param>
-          <param name="blending_time">0.004</param>
-          <param name="realtime_priority">1</param>
+          <param name="ip_address">${ip_address}</param>
+          <param name="port">${port}</param>
+          <param name="session_id">${session_id}</param>
         </xacro:unless>
       </hardware>

Commit message: Added IO state and command interfaces

File: kassow_kord_bringup/urdf/kassow_kord.ros2_control.xacro (robot description, xacro)
@@ -90,4 +90,65 @@
         <state_interface name="effort"/>
       </joint>
+      <xacro:macro name="io_state_interface" params="name io_type index data_type:=bool">
+        <state_interface name="${name}" data_type="${data_type}">
+          <param name="io_type">${io_type}</param>
+           <param name="io_type">${index}</param>
+        </state_interface>
+      </xacro:macro>
+      <gpio name="kassow_digital_IOs">
+        <!-- Digital Inputs DI01 to DI08 Safe Inputs, DI09 to DI16 Quadrature Inputs-->
+        <io_state_interface name="${prefix}_digital_input_1" io_type="DI" index="1"/>
+        <io_state_interface name="${prefix}_digital_input_2" io_type="DI" index="2"/>
+        <io_state_interface name="${prefix}_digital_input_3" io_type="DI" index="3"/>
+        <io_state_interface name="${prefix}_digital_input_4" io_type="DI" index="4"/>
+        <io_state_interface name="${prefix}_digital_input_5" io_type="DI" index="5"/>
+        <io_state_interface name="${prefix}_digital_input_6" io_type="DI" index="6"/>
+        <io_state_interface name="${prefix}_digital_input_7" io_type="DI" index="7"/>
+        <io_state_interface name="${prefix}_digital_input_8" io_type="DI" index="8"/>
+        <io_state_interface name="${prefix}_digital_input_9" io_type="DI" index="9"/>
+        <io_state_interface name="${prefix}_digital_input_10" io_type="DI" index="10"/>
+        <io_state_interface name="${prefix}_digital_input_11" io_type="DI" index="11"/>
+        <io_state_interface name="${prefix}_digital_input_12" io_type="DI" index="12"/>
+        <io_state_interface name="${prefix}_digital_input_13" io_type="DI" index="13"/>
+        <io_state_interface name="${prefix}_digital_input_14" io_type="DI" index="14"/>
+        <io_state_interface name="${prefix}_digital_input_15" io_type="DI" index="15"/>
+        <io_state_interface name="${prefix}_digital_input_16" io_type="DI" index="16"/>
+        <!-- Digital Outputs-->
+        <!-- Digital Relays RELAY1 - RELAY4 -->
+        <!-- <command_interface name="${prefix}_digital_relay_1" data_type="bool"/>
+        <command_interface name="${prefix}_digital_relay_2" data_type="bool"/>
+        <command_interface name="${prefix}_digital_relay_3" data_type="bool"/>
+        <command_interface name="${prefix}_digital_relay_4" data_type="bool"/>
+        <io_state_interface name="${prefix}_digital_relay_1" io_type="RELAY" index="1"/>
+        <io_state_interface name="${prefix}_digital_relay_2" io_type="RELAY" index="2"/>
+        <io_state_interface name="${prefix}_digital_relay_3" io_type="RELAY" index="3"/>
+        <io_state_interface name="${prefix}_digital_relay_4" io_type="RELAY" index="4"/> -->
+        <!-- Digital IO Board DO1 - DO8 -->
+        <!-- <command_interface name="${prefix}_digital_output_1" data_type="bool"/>
+        <command_interface name="${prefix}_digital_output_2" data_type="bool"/>
+        <command_interface name="${prefix}_digital_output_3" data_type="bool"/>
+        <command_interface name="${prefix}_digital_output_4" data_type="bool"/>
+        <command_interface name="${prefix}_digital_output_5" data_type="bool"/>
+        <command_interface name="${prefix}_digital_output_6" data_type="bool"/>
+        <command_interface name="${prefix}_digital_output_7" data_type="bool"/>
+        <command_interface name="${prefix}_digital_output_8" data_type="bool"/>
+        <io_state_interface name="${prefix}_digital_output_1" io_type="DO" index="1"/>
+        <io_state_interface name="${prefix}_digital_output_2" io_type="DO" index="2"/>
+        <io_state_interface name="${prefix}_digital_output_3" io_type="DO" index="3"/>
+        <io_state_interface name="${prefix}_digital_output_4" io_type="DO" index="4"/>
+        <io_state_interface name="${prefix}_digital_output_5" io_type="DO" index="5"/>
+        <io_state_interface name="${prefix}_digital_output_6" io_type="DO" index="6"/>
+        <io_state_interface name="${prefix}_digital_output_7" io_type="DO" index="7"/>
+        <io_state_interface name="${prefix}_digital_output_8" io_type="DO" index="8"/> -->
+        <!-- Digital IO ToolB TB1 - TB4 -->
+        <!-- <command_interface name="${prefix}_digital_tb_1" data_type="bool"/>
+        <command_interface name="${prefix}_digital_tb_2" data_type="bool"/>
+        <command_interface name="${prefix}_digital_tb_3" data_type="bool"/>
+        <command_interface name="${prefix}_digital_tb_4" data_type="bool"/>
+        <io_state_interface name="${prefix}_digital_tb_1" io_type="TB" index="1"/>
+        <io_state_interface name="${prefix}_digital_tb_2" io_type="TB" index="2"/>
+        <io_state_interface name="${prefix}_digital_tb_3" io_type="TB" index="3"/>
+        <io_state_interface name="${prefix}_digital_tb_4" io_type="TB" index="4"/> -->
+      </gpio>
     </ros2_control>
   </xacro:macro>

Commit message: Moved io_state macro to separate file and modified param names

File: kassow_kord_bringup/urdf/kassow_kord.ros2_control.xacro (robot description, xacro)
@@ -1,4 +1,5 @@
 <?xml version="1.0"?>
 <robot xmlns:xacro="http://www.ros.org/wiki/xacro">
+  <xacro:include filename="$(find kassow_kord_bringup)/urdf/kassow_kord_interfaces.ros2_control.xacro"/>
   <xacro:macro name="kassow_kord_ros2_control"
               params="name
@@ -90,39 +91,34 @@
         <state_interface name="effort"/>
       </joint>
-      <xacro:macro name="io_state_interface" params="name io_type index data_type:=bool">
-        <state_interface name="${name}" data_type="${data_type}">
-          <param name="io_type">${io_type}</param>
-           <param name="io_type">${index}</param>
-        </state_interface>
-      </xacro:macro>
       <gpio name="kassow_digital_IOs">
         <!-- Digital Inputs DI01 to DI08 Safe Inputs, DI09 to DI16 Quadrature Inputs-->
-        <io_state_interface name="${prefix}_digital_input_1" io_type="DI" index="1"/>
-        <io_state_interface name="${prefix}_digital_input_2" io_type="DI" index="2"/>
-        <io_state_interface name="${prefix}_digital_input_3" io_type="DI" index="3"/>
-        <io_state_interface name="${prefix}_digital_input_4" io_type="DI" index="4"/>
-        <io_state_interface name="${prefix}_digital_input_5" io_type="DI" index="5"/>
-        <io_state_interface name="${prefix}_digital_input_6" io_type="DI" index="6"/>
-        <io_state_interface name="${prefix}_digital_input_7" io_type="DI" index="7"/>
-        <io_state_interface name="${prefix}_digital_input_8" io_type="DI" index="8"/>
-        <io_state_interface name="${prefix}_digital_input_9" io_type="DI" index="9"/>
-        <io_state_interface name="${prefix}_digital_input_10" io_type="DI" index="10"/>
-        <io_state_interface name="${prefix}_digital_input_11" io_type="DI" index="11"/>
-        <io_state_interface name="${prefix}_digital_input_12" io_type="DI" index="12"/>
-        <io_state_interface name="${prefix}_digital_input_13" io_type="DI" index="13"/>
-        <io_state_interface name="${prefix}_digital_input_14" io_type="DI" index="14"/>
-        <io_state_interface name="${prefix}_digital_input_15" io_type="DI" index="15"/>
-        <io_state_interface name="${prefix}_digital_input_16" io_type="DI" index="16"/>
+        <xacro:io_state_interface name="${prefix}_digital_input_1" io_type="input" bit_index="0"/>
+        <xacro:io_state_interface name="${prefix}_digital_input_2" io_type="input" bit_index="1"/>
+        <xacro:io_state_interface name="${prefix}_digital_input_3" io_type="input" bit_index="2"/>
+        <xacro:io_state_interface name="${prefix}_digital_input_4" io_type="input" bit_index="3"/>
+        <xacro:io_state_interface name="${prefix}_digital_input_5" io_type="input" bit_index="4"/>
+        <xacro:io_state_interface name="${prefix}_digital_input_6" io_type="input" bit_index="5"/>
+        <xacro:io_state_interface name="${prefix}_digital_input_7" io_type="input" bit_index="6"/>
+        <xacro:io_state_interface name="${prefix}_digital_input_8" io_type="input" bit_index="7"/>
+        <xacro:io_state_interface name="${prefix}_digital_input_9" io_type="input" bit_index="8"/>
+        <xacro:io_state_interface name="${prefix}_digital_input_10" io_type="input" bit_index="9"/>
+        <xacro:io_state_interface name="${prefix}_digital_input_11" io_type="input" bit_index="10"/>
+        <xacro:io_state_interface name="${prefix}_digital_input_12" io_type="input" bit_index="11"/>
+        <xacro:io_state_interface name="${prefix}_digital_input_13" io_type="input" bit_index="12"/>
+        <xacro:io_state_interface name="${prefix}_digital_input_14" io_type="input" bit_index="13"/>
+        <xacro:io_state_interface name="${prefix}_digital_input_15" io_type="input" bit_index="14"/>
+        <xacro:io_state_interface name="${prefix}_digital_input_16" io_type="input" bit_index="15"/>
         <!-- Digital Outputs-->
-        <!-- Digital Relays RELAY1 - RELAY4 -->
+         <!-- Bit indexes are defined according to the convention used in Kassow API-->
+        <!-- Digital Relays RELAY1 - RELAY4 - Bit indexes 0 - 3 -->
         <!-- <command_interface name="${prefix}_digital_relay_1" data_type="bool"/>
         <command_interface name="${prefix}_digital_relay_2" data_type="bool"/>
         <command_interface name="${prefix}_digital_relay_3" data_type="bool"/>
-        <command_interface name="${prefix}_digital_relay_4" data_type="bool"/>
-        <io_state_interface name="${prefix}_digital_relay_1" io_type="RELAY" index="1"/>
-        <io_state_interface name="${prefix}_digital_relay_2" io_type="RELAY" index="2"/>
-        <io_state_interface name="${prefix}_digital_relay_3" io_type="RELAY" index="3"/>
-        <io_state_interface name="${prefix}_digital_relay_4" io_type="RELAY" index="4"/> -->
-        <!-- Digital IO Board DO1 - DO8 -->
+        <command_interface name="${prefix}_digital_relay_4" data_type="bool"/> -->
+        <!-- <xacro:io_state_interface name="${prefix}_digital_relay_1" io_type="RELAY" bit_index="0"/>
+        <xacro:io_state_interface name="${prefix}_digital_relay_2" io_type="RELAY" bit_index="1"/>
+        <xacro:io_state_interface name="${prefix}_digital_relay_3" io_type="RELAY" bit_index="2"/>
+        <xacro:io_state_interface name="${prefix}_digital_relay_4" io_type="RELAY" bit_index="3"/> -->
+        <!-- Digital IO Board DO1 - DO8 - Bit indexes 4 - 11 -->
         <!-- <command_interface name="${prefix}_digital_output_1" data_type="bool"/>
         <command_interface name="${prefix}_digital_output_2" data_type="bool"/>
@@ -132,22 +128,22 @@
         <command_interface name="${prefix}_digital_output_6" data_type="bool"/>
         <command_interface name="${prefix}_digital_output_7" data_type="bool"/>
-        <command_interface name="${prefix}_digital_output_8" data_type="bool"/>
-        <io_state_interface name="${prefix}_digital_output_1" io_type="DO" index="1"/>
-        <io_state_interface name="${prefix}_digital_output_2" io_type="DO" index="2"/>
-        <io_state_interface name="${prefix}_digital_output_3" io_type="DO" index="3"/>
-        <io_state_interface name="${prefix}_digital_output_4" io_type="DO" index="4"/>
-        <io_state_interface name="${prefix}_digital_output_5" io_type="DO" index="5"/>
-        <io_state_interface name="${prefix}_digital_output_6" io_type="DO" index="6"/>
-        <io_state_interface name="${prefix}_digital_output_7" io_type="DO" index="7"/>
-        <io_state_interface name="${prefix}_digital_output_8" io_type="DO" index="8"/> -->
-        <!-- Digital IO ToolB TB1 - TB4 -->
+        <command_interface name="${prefix}_digital_output_8" data_type="bool"/> -->
+        <!-- <xacro:io_state_interface name="${prefix}_digital_output_1" io_type="DO" bit_index="4"/>
+        <xacro:io_state_interface name="${prefix}_digital_output_2" io_type="DO" bit_index="5"/>
+        <xacro:io_state_interface name="${prefix}_digital_output_3" io_type="DO" bit_index="6"/>
+        <xacro:io_state_interface name="${prefix}_digital_output_4" io_type="DO" bit_index="7"/>
+        <xacro:io_state_interface name="${prefix}_digital_output_5" io_type="DO" bit_index="8"/>
+        <xacro:io_state_interface name="${prefix}_digital_output_6" io_type="DO" bit_index="9"/>
+        <xacro:io_state_interface name="${prefix}_digital_output_7" io_type="DO" bit_index="10"/>
+        <xacro:io_state_interface name="${prefix}_digital_output_8" io_type="DO" bit_index="11"/> -->
+        <!-- Digital IO ToolB TB1 - TB4 - Bit indexes 12 - 15 -->
         <!-- <command_interface name="${prefix}_digital_tb_1" data_type="bool"/>
         <command_interface name="${prefix}_digital_tb_2" data_type="bool"/>
         <command_interface name="${prefix}_digital_tb_3" data_type="bool"/>
-        <command_interface name="${prefix}_digital_tb_4" data_type="bool"/>
-        <io_state_interface name="${prefix}_digital_tb_1" io_type="TB" index="1"/>
-        <io_state_interface name="${prefix}_digital_tb_2" io_type="TB" index="2"/>
-        <io_state_interface name="${prefix}_digital_tb_3" io_type="TB" index="3"/>
-        <io_state_interface name="${prefix}_digital_tb_4" io_type="TB" index="4"/> -->
+        <command_interface name="${prefix}_digital_tb_4" data_type="bool"/> -->
+        <!-- <xacro:io_state_interface name="${prefix}_digital_tb_1" io_type="TB" bit_index="12"/>
+        <xacro:io_state_interface name="${prefix}_digital_tb_2" io_type="TB" bit_index="13"/>
+        <xacro:io_state_interface name="${prefix}_digital_tb_3" io_type="TB" bit_index="14"/>
+        <xacro:io_state_interface name="${prefix}_digital_tb_4" io_type="TB" bit_index="15"/> -->
       </gpio>
     </ros2_control>
