Commit message: Add IO command interfaces macro

File: kassow_kord_bringup/urdf/kassow_kord.ros2_control.xacro (robot description, xacro)
@@ -112,8 +112,8 @@
          <!-- Bit indexes are defined according to the convention used in Kassow API-->
         <!-- Digital Relays RELAY1 - RELAY4 - Bit indexes 0 - 3 -->
-        <!-- <command_interface name="${prefix}_digital_relay_1" data_type="bool"/>
-        <command_interface name="${prefix}_digital_relay_2" data_type="bool"/>
-        <command_interface name="${prefix}_digital_relay_3" data_type="bool"/>
-        <command_interface name="${prefix}_digital_relay_4" data_type="bool"/> -->
+        <xacro:io_command_interface name="${prefix}_digital_relay_1" io_type="output" bit_index="0"/>
+        <xacro:io_command_interface name="${prefix}_digital_relay_2" io_type="output" bit_index="1"/>
+        <xacro:io_command_interface name="${prefix}_digital_relay_3" io_type="output" bit_index="2"/>
+        <xacro:io_command_interface name="${prefix}_digital_relay_4" io_type="output" bit_index="3"/>
         <xacro:io_state_interface name="${prefix}_digital_relay_1" io_type="output" bit_index="0"/>
         <xacro:io_state_interface name="${prefix}_digital_relay_2" io_type="output" bit_index="1"/>
@@ -121,12 +121,12 @@
         <xacro:io_state_interface name="${prefix}_digital_relay_4" io_type="output" bit_index="3"/>
         <!-- Digital IO Board DO1 - DO8 - Bit indexes 4 - 11 -->
-        <!-- <command_interface name="${prefix}_digital_output_1" data_type="bool"/>
-        <command_interface name="${prefix}_digital_output_2" data_type="bool"/>
-        <command_interface name="${prefix}_digital_output_3" data_type="bool"/>
-        <command_interface name="${prefix}_digital_output_4" data_type="bool"/>
-        <command_interface name="${prefix}_digital_output_5" data_type="bool"/>
-        <command_interface name="${prefix}_digital_output_6" data_type="bool"/>
-        <command_interface name="${prefix}_digital_output_7" data_type="bool"/>
-        <command_interface name="${prefix}_digital_output_8" data_type="bool"/> -->
+        <xacro:io_command_interface name="${prefix}_digital_output_1" io_type="output" bit_index="4"/>
+        <xacro:io_command_interface name="${prefix}_digital_output_2" io_type="output" bit_index="5"/>
+        <xacro:io_command_interface name="${prefix}_digital_output_3" io_type="output" bit_index="6"/>
+        <xacro:io_command_interface name="${prefix}_digital_output_4" io_type="output" bit_index="7"/>
+        <xacro:io_command_interface name="${prefix}_digital_output_5" io_type="output" bit_index="8"/>
+        <xacro:io_command_interface name="${prefix}_digital_output_6" io_type="output" bit_index="9"/>
+        <xacro:io_command_interface name="${prefix}_digital_output_7" io_type="output" bit_index="10"/>
+        <xacro:io_command_interface name="${prefix}_digital_output_8" io_type="output" bit_index="11"/>
         <xacro:io_state_interface name="${prefix}_digital_output_1" io_type="output" bit_index="4"/>
         <xacro:io_state_interface name="${prefix}_digital_output_2" io_type="output" bit_index="5"/>
@@ -138,8 +138,8 @@
         <xacro:io_state_interface name="${prefix}_digital_output_8" io_type="output" bit_index="11"/>
         <!-- Digital IO ToolB TB1 - TB4 - Bit indexes 12 - 15 -->
-        <!-- <command_interface name="${prefix}_digital_tb_1" data_type="bool"/>
-        <command_interface name="${prefix}_digital_tb_2" data_type="bool"/>
-        <command_interface name="${prefix}_digital_tb_3" data_type="bool"/>
-        <command_interface name="${prefix}_digital_tb_4" data_type="bool"/> -->
+        <xacro:io_command_interface name="${prefix}_digital_tb_1" io_type="output" bit_index="12"/>
+        <xacro:io_command_interface name="${prefix}_digital_tb_2" io_type="output" bit_index="13"/>
+        <xacro:io_command_interface name="${prefix}_digital_tb_3" io_type="output" bit_index="14"/>
+        <xacro:io_command_interface name="${prefix}_digital_tb_4" io_type="output" bit_index="15"/>
         <xacro:io_state_interface name="${prefix}_digital_tb_1" io_type="output" bit_index="12"/>
         <xacro:io_state_interface name="${prefix}_digital_tb_2" io_type="output" bit_index="13"/>

File: kassow_kord_bringup/urdf/kassow_kord_interfaces.ros2_control.xacro (robot description, xacro)
@@ -7,3 +7,9 @@
     </state_interface>
   </xacro:macro>
+  <xacro:macro name="io_command_interface" params="name io_type bit_index data_type:=bool">
+    <command_interface name="${name}" data_type="${data_type}">
+      <param name="io_type">${io_type}</param>
+      <param name="bit_index">${bit_index}</param>
+    </command_interface>
+  </xacro:macro>
 </robot>
