Commit message: Corrected data_type to double

File: kassow_kord_bringup/urdf/kassow_kord_interfaces.ros2_control.xacro (robot description, xacro)
@@ -1,5 +1,5 @@
 <?xml version="1.0"?>
 <robot xmlns:xacro="http://www.ros.org/wiki/xacro">
-  <xacro:macro name="io_state_interface" params="name io_type bit_index data_type:=bool">
+  <xacro:macro name="io_state_interface" params="name io_type bit_index data_type:=double">
     <state_interface name="${name}" data_type="${data_type}">
       <param name="io_type">${io_type}</param>
@@ -7,5 +7,5 @@
     </state_interface>
   </xacro:macro>
-  <xacro:macro name="io_command_interface" params="name io_type bit_index data_type:=bool">
+  <xacro:macro name="io_command_interface" params="name io_type bit_index data_type:=double">
     <command_interface name="${name}" data_type="${data_type}">
       <param name="io_type">${io_type}</param>
