Commit message: fix rounding issues

File: kassow_kord_description/kr810/urdf/kr810_description.urdf.xacro (robot description, xacro)
@@ -282,5 +282,5 @@
     <axis xyz="0 0 1"/>
     <dynamics damping="${joints_damping}"/>
-    <limit effort="204" velocity="${225/180*pi}" lower="${-2*pi}" upper="${2*pi}"/>
+    <limit effort="204" velocity="${radians(225)}" lower="${-2*pi}" upper="${2*pi}"/>
   </joint>
   <xacro:property name="joint1_xoffset"  value="${  50.0 * scale}" />
@@ -293,5 +293,5 @@
     <axis xyz="0 1 0"/>
     <dynamics damping="${joints_damping}"/>
-    <limit effort="204" velocity="${225/180*pi}" lower="${-70.0 * pi_per_deg}" upper="${(180/180)*pi}"/>
+    <limit effort="204" velocity="${radians(225)}" lower="-${radians(70.0)}" upper="${pi}"/>
   </joint>
   <xacro:property name="jointPL2_xoffset"  value="${  -50.0 * scale}" />
@@ -308,5 +308,5 @@
     <axis xyz="0 0 1"/>
     <dynamics damping="${joints_damping}"/>
-    <limit effort="85" velocity="${225/180*pi}" lower="${-2*pi}" upper="${2*pi}"/>
+    <limit effort="85" velocity="${radians(225)}" lower="${-2*pi}" upper="${2*pi}"/>
   </joint>
   <xacro:property name="joint3_xoffset"  value="${ 40.0 * scale}" />
@@ -319,5 +319,5 @@
     <axis xyz="0 1 0"/>
     <dynamics damping="${joints_damping}"/>
-    <limit effort="85" velocity="${225/180*pi}" lower="${-70.0 * pi_per_deg}" upper="${(180/180)*pi}"/>
+    <limit effort="85" velocity="${radians(225)}" lower="-${radians(70.0)}" upper="${pi}"/>
   </joint>
   <xacro:property name="jointPL4_xoffset"  value="${ -40.0 * scale}" />
@@ -335,5 +335,5 @@
     <axis xyz="0 0 1"/>
     <dynamics damping="${joints_damping}"/>
-    <limit effort="51" velocity="${225/180*pi}" lower="${-2*pi}" upper="${2*pi}"/>
+    <limit effort="51" velocity="${radians(225)}" lower="${-2*pi}" upper="${2*pi}"/>
   </joint>
   <xacro:property name="joint5_zoffset"  value="${ 103.5 * scale}" />
@@ -344,5 +344,5 @@
     <axis xyz="0 1 0"/>
     <dynamics damping="${joints_damping}"/>
-    <limit effort="51" velocity="${225/180*pi}" lower="${-2*pi}" upper="${2*pi}"/>
+    <limit effort="51" velocity="${radians(225)}" lower="${-2*pi}" upper="${2*pi}"/>
   </joint>
   <xacro:property name="jointPL6_yoffset"  value="${ 111.0 * scale}" />
@@ -359,5 +359,5 @@
     <axis xyz="0 0 1"/>
     <dynamics damping="${joints_damping}"/>
-    <limit effort="51" velocity="${225/180*pi}" lower="${-2*pi}" upper="${2*pi}"/>
+    <limit effort="51" velocity="${radians(225)}" lower="${-2*pi}" upper="${2*pi}"/>
   </joint>
   </xacro:macro>

Commit message: Correct effort limits.

File: kassow_kord_description/kr810/urdf/kr810_description.urdf.xacro (robot description, xacro)
@@ -282,5 +282,5 @@
     <axis xyz="0 0 1"/>
     <dynamics damping="${joints_damping}"/>
-    <limit effort="204" velocity="${radians(225)}" lower="${-2*pi}" upper="${2*pi}"/>
+    <limit effort="60" velocity="${radians(225)}" lower="${-2*pi}" upper="${2*pi}"/>
   </joint>
   <xacro:property name="joint1_xoffset"  value="${  50.0 * scale}" />
@@ -293,5 +293,5 @@
     <axis xyz="0 1 0"/>
     <dynamics damping="${joints_damping}"/>
-    <limit effort="204" velocity="${radians(225)}" lower="-${radians(70.0)}" upper="${pi}"/>
+    <limit effort="60" velocity="${radians(225)}" lower="-${radians(70.0)}" upper="${pi}"/>
   </joint>
   <xacro:property name="jointPL2_xoffset"  value="${  -50.0 * scale}" />
@@ -308,5 +308,5 @@
     <axis xyz="0 0 1"/>
     <dynamics damping="${joints_damping}"/>
-    <limit effort="85" velocity="${radians(225)}" lower="${-2*pi}" upper="${2*pi}"/>
+    <limit effort="40" velocity="${radians(225)}" lower="${-2*pi}" upper="${2*pi}"/>
   </joint>
   <xacro:property name="joint3_xoffset"  value="${ 40.0 * scale}" />
@@ -319,5 +319,5 @@
     <axis xyz="0 1 0"/>
     <dynamics damping="${joints_damping}"/>
-    <limit effort="85" velocity="${radians(225)}" lower="-${radians(70.0)}" upper="${pi}"/>
+    <limit effort="40" velocity="${radians(225)}" lower="-${radians(70.0)}" upper="${pi}"/>
   </joint>
   <xacro:property name="jointPL4_xoffset"  value="${ -40.0 * scale}" />
@@ -335,5 +335,5 @@
     <axis xyz="0 0 1"/>
     <dynamics damping="${joints_damping}"/>
-    <limit effort="51" velocity="${radians(225)}" lower="${-2*pi}" upper="${2*pi}"/>
+    <limit effort="20" velocity="${radians(225)}" lower="${-2*pi}" upper="${2*pi}"/>
   </joint>
   <xacro:property name="joint5_zoffset"  value="${ 103.5 * scale}" />
@@ -344,5 +344,5 @@
     <axis xyz="0 1 0"/>
     <dynamics damping="${joints_damping}"/>
-    <limit effort="51" velocity="${radians(225)}" lower="${-2*pi}" upper="${2*pi}"/>
+    <limit effort="20" velocity="${radians(225)}" lower="${-2*pi}" upper="${2*pi}"/>
   </joint>
   <xacro:property name="jointPL6_yoffset"  value="${ 111.0 * scale}" />
@@ -359,5 +359,5 @@
     <axis xyz="0 0 1"/>
     <dynamics damping="${joints_damping}"/>
-    <limit effort="51" velocity="${radians(225)}" lower="${-2*pi}" upper="${2*pi}"/>
+    <limit effort="20" velocity="${radians(225)}" lower="${-2*pi}" upper="${2*pi}"/>
   </joint>
   </xacro:macro>
