Commit message: description: standardize mesh files

File: kassow_kord_description/kr810/urdf/kr810_description.urdf.xacro (robot description, xacro)
@@ -1,5 +1,5 @@
 <?xml version="1.0" ?>
 <robot name="kr2_robot_a810" model="a810" model-revision="051020-0" mechanical-revision="5" features="TIO" xmlns:xacro="http://www.ros.org/wiki/xacro">
-  <xacro:macro name="kr810_description" params="prefix parent *origin">
+  <xacro:macro name="kassow_robot" params="prefix parent *origin">
   <!-- globals -->
   <xacro:property name="joints_damping" value="0.1" />
@@ -67,5 +67,5 @@
       rpy="0 0 0"
       color="0.2 0.2 0.2 1"
-      mesh_file="package://kassow_kord_description/kr810/meshes/a810/a810_Base.stl"
+      mesh_file="package://kassow_kord_description/kr810/meshes/collision/a810_Base.stl"
       scale="0.001 0.001 0.001"/>
   </link>
@@ -87,5 +87,5 @@
       rpy="0 0 0"
       color="0.2 0.2 0.2 1"
-      mesh_file="package://kassow_kord_description/kr810/meshes/a810/a810_Link2.stl"
+      mesh_file="package://kassow_kord_description/kr810/meshes/collision/a810_Link2.stl"
       scale="0.001 0.001 0.001"/>
   </link>
@@ -122,5 +122,5 @@
       rpy="-${pi/2} 0 -${pi/2}"
       color="0.2 0.2 0.2 1"
-      mesh_file="package://kassow_kord_description/kr810/meshes/a810/a810_Link3.stl"
+      mesh_file="package://kassow_kord_description/kr810/meshes/collision/a810_Link3.stl"
       scale="0.001 0.001 0.001"/>
   </link>
@@ -143,5 +143,5 @@
       rpy="${pi/2} 0 -${pi/2}"
       color="0.2 0.2 0.2 1"
-      mesh_file="package://kassow_kord_description/kr810/meshes/a810/a810_Link4.stl"
+      mesh_file="package://kassow_kord_description/kr810/meshes/collision/a810_Link4.stl"
       scale="0.001 0.001 0.001"/>
   </link>
@@ -178,5 +178,5 @@
       rpy="-${pi/2} 0 ${pi/2}"
       color="0.2 0.2 0.2 1"
-      mesh_file="package://kassow_kord_description/kr810/meshes/a810/a810_Link5.stl"
+      mesh_file="package://kassow_kord_description/kr810/meshes/collision/a810_Link5.stl"
       scale="0.001 0.001 0.001"/>
   </link>
@@ -196,5 +196,5 @@
       rpy="0 0 -${pi/2}"
       color="0.2 0.2 0.2 1"
-      mesh_file="package://kassow_kord_description/kr810/meshes/a810/a810_Link6.stl"
+      mesh_file="package://kassow_kord_description/kr810/meshes/collision/a810_Link6.stl"
       scale="0.001 0.001 0.001"/>
   </link>
@@ -231,5 +231,5 @@
       rpy="0 0 0"
       color="0.2 0.2 0.2 1"
-      mesh_file="package://kassow_kord_description/kr810/meshes/a810/a810_Link7.stl"
+      mesh_file="package://kassow_kord_description/kr810/meshes/collision/a810_Link7.stl"
       scale="0.001 0.001 0.001"/>
   </link>
@@ -251,5 +251,5 @@
       rpy="0 0 0"
       color="0.8 0.8 0.8 1"
-      mesh_file="package://kassow_kord_description/kr810/meshes/a810/a810_ToolIO.stl"
+      mesh_file="package://kassow_kord_description/kr810/meshes/collision/a810_ToolIO.stl"
       scale="0.001 0.001 0.001"/>
   </link>
