Commit message: fix collisions and cleanup urdf

File: kassow_kord_bringup/srdf/kassow_kord.srdf.xacro (robot description, xacro)
@@ -19,10 +19,12 @@
     <disable_collisions link1="base" link2="link1" reason="Adjacent" />
     <disable_collisions link1="link1" link2="linkJ2" reason="Adjacent" />
-    <disable_collisions link1="linkJ2" link2="link2" reason="Never" />
-    <disable_collisions link1="link2" link2="link3" reason="Never" />
-    <disable_collisions link1="link3" link2="linkJ4" reason="Never" />
+    <disable_collisions link1="link1" link2="link2" reason="Adjacent" />
+    <disable_collisions link1="linkJ2" link2="link2" reason="Adjacent" />
+    <disable_collisions link1="link2" link2="link3" reason="Adjacent" />
+    <disable_collisions link1="link3" link2="linkJ4" reason="Adjacent" />
     <disable_collisions link1="linkJ4" link2="link4" reason="Adjacent" />
     <disable_collisions link1="link4" link2="link5" reason="Adjacent" />
-    <disable_collisions link1="link5" link2="linkJ6" reason="Never" />
+    <disable_collisions link1="link5" link2="linkJ6" reason="Adjacent" />
+    <disable_collisions link1="link5" link2="link6" reason="Adjacent" />
     <disable_collisions link1="linkJ6" link2="link6" reason="Adjacent" />
     <disable_collisions link1="link6" link2="end_effector" reason="Adjacent" />

File: kassow_kord_description/kr810/urdf/kr810_description.urdf.xacro (robot description, xacro)
@@ -20,5 +20,4 @@
   <!-- globals -->
   <xacro:property name="joints_damping" value="0.1" />
-  <!-- links -->
   <!-- all dimensions should be input as measured in the drawing in mm and
        converted to real dimensions by multiplying with the scale property -->
@@ -28,11 +27,4 @@
   <xacro:property name="mass_multiplier" value="1.0" />
   <xacro:macro name="cylinder_inertia" params="mass radius length">
-      <!--      <inertia ixx="${mass/12*(3*radius*radius+3*length*length)}"
-               ixy="0.0"
-               ixz="0.0"
-               iyy="${mass/12*(3*radius*radius+3*length*length)}"
-               iyz="0.0"
-               izz="${mass*radius*radius/2}"/>
-       -->
       <inertia ixx="0.003"
                ixy="0.0"
@@ -57,4 +49,21 @@
       </collision>
   </xacro:macro>
+  <xacro:macro name="visual_and_collision_mesh" params="xyz rpy color mesh_file scale">
+    <visual>
+      <origin rpy="${rpy}" xyz="${xyz}" />
+      <geometry>
+        <mesh filename="${mesh_file}" scale="${scale}"/>
+      </geometry>
+      <material name="">
+        <color rgba="${color}" />
+      </material>
+    </visual>
+    <collision>
+      <origin rpy="${rpy}" xyz="${xyz}" />
+      <geometry>
+        <mesh filename="${mesh_file}" scale="${scale}"/>
+      </geometry>
+    </collision>
+  </xacro:macro>
   <link name="world"/>
   <link name="base">
@@ -64,16 +73,4 @@
     <xacro:property name="base_inner_height" value="${ 15 * scale}" />
     <xacro:property name="base_mass"         value="0.6" />
-    <!--
-    <xacro:visual_and_collision rpy="0 0 0"
-                                xyz="0 0 ${base_outer_height / 2}"
-                                material="dark_gray">
-      <cylinder length="${base_outer_height}" radius="${base_outer_radius}"/>
-    </xacro:visual_and_collision>
-    <xacro:visual_and_collision rpy="0 0 0"
-                                xyz="0 0 ${base_outer_height + base_inner_height/2}"
-                                material="dark_gray">
-      <cylinder length="${base_inner_height}" radius="${base_inner_radius}"/>
-    </xacro:visual_and_collision>
-    -->
     <inertial>
       <origin rpy="0 0 0" xyz="0 0 0"/>
@@ -83,13 +80,10 @@
                               length="${base_inner_height+base_outer_height}" />
     </inertial>
-    <visual>
-        <origin xyz="0 0 0" rpy="0 0 0" />
-        <geometry>
-          <mesh filename="package://kassow_kord_description/kr810/meshes/a810/a810_Base.stl" scale="0.001 0.001 0.001"/>
-        </geometry>
-        <material name="">
-          <color rgba="0.2 0.2 0.2 1" />
-        </material>
-    </visual>
+    <xacro:visual_and_collision_mesh
+      xyz="0 0 0"
+      rpy="0 0 0"
+      color="0.2 0.2 0.2 1"
+      mesh_file="package://kassow_kord_description/kr810/meshes/a810/a810_Base.stl"
+      scale="0.001 0.001 0.001"/>
   </link>
   <link name="link1">
@@ -99,37 +93,17 @@
     <xacro:property name="link1_hinge_radius"  value="${  57.5 * scale}" />
     <xacro:property name="link1_mass"   value="4.58" />
-    <!--
-    <xacro:visual_and_collision rpy="0 0 0"
-                                xyz="0 0 ${link1_length/2 - 25 * scale}"
-                                material="gray">
-      <cylinder length="${link1_length - 50 * scale}" radius="${link1_radius}"/>
-    </xacro:visual_and_collision>
-    <xacro:visual_and_collision rpy="${pi/2} 0 0"
-                                xyz="${50 * scale} ${20 * scale} ${link1_length}"
-                                material="gray">
-      <cylinder length="${link1_radius * 1.7}" radius="${link1_radius}"/>
-    </xacro:visual_and_collision>
-    <xacro:visual_and_collision rpy="0 ${pi/4} 0"
-                                xyz="${20 * scale} ${+8 * scale} ${200 * scale}"
-                                material="light_gray">
-      <cylinder length="${90 * scale}" radius="${50 * scale}"/>
-    </xacro:visual_and_collision>
-    -->
     <inertial>
       <origin rpy="0 0 0" xyz="0 0 ${link1_length/2}"/>
       <mass value="${link1_mass*mass_multiplier}"/>
-            <xacro:cylinder_inertia mass="${link1_mass}"
-                                    radius="${link1_radius}"
-                                    length="${link1_length}" />
-    </inertial>
-    <visual>
-        <origin xyz="0 0 0.169" rpy="0 0 0" />
-        <geometry>
-          <mesh filename="package://kassow_kord_description/kr810/meshes/a810/a810_Link2.stl" scale="0.001 0.001 0.001"/>
-        </geometry>
-        <material name="">
-          <color rgba="0.2 0.2 0.2 1" />
-        </material>
-    </visual>
+      <xacro:cylinder_inertia mass="${link1_mass}"
+                              radius="${link1_radius}"
+                              length="${link1_length}"/>
+    </inertial>
+    <xacro:visual_and_collision_mesh
+      xyz="0 0 0.169"
+      rpy="0 0 0"
+      color="0.2 0.2 0.2 1"
+      mesh_file="package://kassow_kord_description/kr810/meshes/a810/a810_Link2.stl"
+      scale="0.001 0.001 0.001"/>
   </link>
   <link name="linkJ2">
@@ -161,13 +135,10 @@
                               length="${link2_length}" />
     </inertial>
-    <visual>
-        <origin xyz="0.049 0 0" rpy="-${pi/2} 0 -${pi/2}" />
-        <geometry>
-          <mesh filename="package://kassow_kord_description/kr810/meshes/a810/a810_Link3.stl" scale="0.001 0.001 0.001"/>
-        </geometry>
-        <material name="">
-          <color rgba="0.2 0.2 0.2 1" />
-        </material>
-    </visual>
+    <xacro:visual_and_collision_mesh
+      xyz="0.049 0 0"
+      rpy="-${pi/2} 0 -${pi/2}"
+      color="0.2 0.2 0.2 1"
+      mesh_file="package://kassow_kord_description/kr810/meshes/a810/a810_Link3.stl"
+      scale="0.001 0.001 0.001"/>
   </link>
   <link name="link3">
@@ -185,13 +156,10 @@
                               length="${link3_length}" />
     </inertial>
-    <visual>
-        <origin xyz="-0.05 -0.0 0.315" rpy="${pi/2} 0 -${pi/2}" />
-        <geometry>
-          <mesh filename="package://kassow_kord_description/kr810/meshes/a810/a810_Link4.stl" scale="0.001 0.001 0.001"/>
-        </geometry>
-        <material name="">
-          <color rgba="0.2 0.2 0.2 1" />
-        </material>
-    </visual>
+    <xacro:visual_and_collision_mesh
+      xyz="-0.05 -0.0 0.315"
+      rpy="${pi/2} 0 -${pi/2}"
+      color="0.2 0.2 0.2 1"
+      mesh_file="package://kassow_kord_description/kr810/meshes/a810/a810_Link4.stl"
+      scale="0.001 0.001 0.001"/>
   </link>
   <link name="linkJ4">
@@ -223,13 +191,10 @@
                               length="${link4_length}" />
     </inertial>
-    <visual>
-        <origin xyz="0.04 0.0005 0.0" rpy="-${pi/2} 0 ${pi/2}" />
-        <geometry>
-          <mesh filename="package://kassow_kord_description/kr810/meshes/a810/a810_Link5.stl" scale="0.001 0.001 0.001"/>
-        </geometry>
-        <material name="">
-          <color rgba="0.2 0.2 0.2 1" />
-        </material>
-    </visual>
+    <xacro:visual_and_collision_mesh
+      xyz="0.04 0.0005 0.0"
+      rpy="-${pi/2} 0 ${pi/2}"
+      color="0.2 0.2 0.2 1"
+      mesh_file="package://kassow_kord_description/kr810/meshes/a810/a810_Link5.stl"
+      scale="0.001 0.001 0.001"/>
   </link>
   <link name="link5">
@@ -244,13 +209,10 @@
                               length="${link5_length}" />
     </inertial>
-    <visual>
-        <origin xyz="0.0 0.002 0.1035" rpy="0 0 -${pi/2}" />
-        <geometry>
-          <mesh filename="package://kassow_kord_description/kr810/meshes/a810/a810_Link6.stl" scale="0.001 0.001 0.001"/>
-        </geometry>
-        <material name="">
-          <color rgba="0.2 0.2 0.2 1" />
-        </material>
-    </visual>
+    <xacro:visual_and_collision_mesh
+      xyz="0.0 0.002 0.1035"
+      rpy="0 0 -${pi/2}"
+      color="0.2 0.2 0.2 1"
+      mesh_file="package://kassow_kord_description/kr810/meshes/a810/a810_Link6.stl"
+      scale="0.001 0.001 0.001"/>
   </link>
   <link name="linkJ6">
@@ -258,5 +220,4 @@
     <xacro:property name="cylinderJ6_height"   value="${ 110.0 * scale}"  />
     <xacro:property name="linkJ6_mass"         value="1.8"   />
-    <!--
     <xacro:visual_and_collision rpy="${pi/2} 0 0"
                                 xyz="0 ${10 * scale} 0"
@@ -264,5 +225,4 @@
       <cylinder length="${cylinderJ6_height * 1.9}" radius="${cylinderJ6_radius}"/>
     </xacro:visual_and_collision>
-    -->
     <inertial>
       <origin rpy="0 0 0" xyz="0 ${4.0 * scale} 0"/>
@@ -284,13 +244,10 @@
                               length="${link6_length}" />
     </inertial>
-    <visual>
-        <origin xyz="0.0 0.0 0.0" rpy="0 0 0" />
-        <geometry>
-          <mesh filename="package://kassow_kord_description/kr810/meshes/a810/a810_Link7.stl" scale="0.001 0.001 0.001"/>
-        </geometry>
-        <material name="">
-          <color rgba="0.2 0.2 0.2 1" />
-        </material>
-    </visual>
+    <xacro:visual_and_collision_mesh
+      xyz="0.0 0.0 0.0"
+      rpy="0 0 0"
+      color="0.2 0.2 0.2 1"
+      mesh_file="package://kassow_kord_description/kr810/meshes/a810/a810_Link7.stl"
+      scale="0.001 0.001 0.001"/>
   </link>
   <link name="end_effector">
@@ -299,14 +256,5 @@
     <xacro:property name="end_effector_inner_radius" value="${ 22.5 * scale}" />
     <xacro:property name="end_effector_inner_length" value="${ 5.0   * scale}" />
-    <xacro:property name="end_effector_mass"         value="0.56"   />
-    <visual>
-        <origin xyz="0.0 -0.0 0.0" rpy="0 0 0" />
-        <geometry>
-          <mesh filename="package://kassow_kord_description/kr810/meshes/a810/a810_ToolIO.stl" scale="0.001 0.001 0.001"/>
-        </geometry>
-        <material name="">
-          <color rgba="0.8 0.8 0.8 1" />
-        </material>
-    </visual>
+    <xacro:property name="end_effector_mass" value="0.56"/>
     <inertial>
       <origin rpy="0 0 0" xyz="0 0 ${-19.7 * scale}"/>
@@ -316,4 +264,10 @@
                               length="${end_effector_outer_length + end_effector_inner_length}" />
     </inertial>
+    <xacro:visual_and_collision_mesh
+      xyz="0.0 -0.0 0.0"
+      rpy="0 0 0"
+      color="0.8 0.8 0.8 1"
+      mesh_file="package://kassow_kord_description/kr810/meshes/a810/a810_ToolIO.stl"
+      scale="0.001 0.001 0.001"/>
   </link>
   <!-- joints -->
@@ -329,5 +283,4 @@
     <dynamics damping="${joints_damping}"/>
     <limit effort="204" velocity="${225/180*pi}" lower="${-2*pi}" upper="${2*pi}"/>
-    <!-- <limit effort="204" velocity="${225/180*pi}" lower="${-122.6 * pi_per_deg}" upper="${127.6 * pi_per_deg}"/> -->
   </joint>
   <xacro:property name="joint1_xoffset"  value="${  50.0 * scale}" />
@@ -341,5 +294,4 @@
     <dynamics damping="${joints_damping}"/>
     <limit effort="204" velocity="${225/180*pi}" lower="${-70.0 * pi_per_deg}" upper="${(180/180)*pi}"/>
-    <!-- <limit effort="204" velocity="${225/180*pi}" lower="${-31.9 * pi_per_deg}" upper="${168.5 * pi_per_deg}"/> -->
   </joint>
   <xacro:property name="jointPL2_xoffset"  value="${  -50.0 * scale}" />
@@ -357,5 +309,4 @@
     <dynamics damping="${joints_damping}"/>
     <limit effort="85" velocity="${225/180*pi}" lower="${-2*pi}" upper="${2*pi}"/>
-    <!--  <limit effort="85" velocity="${225/180*pi}" lower="${-177.6 * pi_per_deg}" upper="${177.6 * pi_per_deg}"/> -->
   </joint>
   <xacro:property name="joint3_xoffset"  value="${ 40.0 * scale}" />
@@ -369,5 +320,4 @@
     <dynamics damping="${joints_damping}"/>
     <limit effort="85" velocity="${225/180*pi}" lower="${-70.0 * pi_per_deg}" upper="${(180/180)*pi}"/>
-    <!-- <limit effort="85" velocity="${225/180*pi}" lower="${-20.6 * pi_per_deg}" upper="${152.1 * pi_per_deg}"/> -->
   </joint>
   <xacro:property name="jointPL4_xoffset"  value="${ -40.0 * scale}" />
@@ -386,5 +336,4 @@
     <dynamics damping="${joints_damping}"/>
     <limit effort="51" velocity="${225/180*pi}" lower="${-2*pi}" upper="${2*pi}"/>
-    <!-- <limit effort="51" velocity="${225/180*pi}" lower="${-177.6 * pi_per_deg}" upper="${177.6 * pi_per_deg}"/> -->
   </joint>
   <xacro:property name="joint5_zoffset"  value="${ 103.5 * scale}" />
@@ -396,5 +345,4 @@
     <dynamics damping="${joints_damping}"/>
     <limit effort="51" velocity="${225/180*pi}" lower="${-2*pi}" upper="${2*pi}"/>
-    <!--    <limit effort="51" velocity="${225/180*pi}" lower="${-177.6 * pi_per_deg}" upper="${177.6 * pi_per_deg}"/> -->
   </joint>
   <xacro:property name="jointPL6_yoffset"  value="${ 111.0 * scale}" />
@@ -412,5 +360,4 @@
     <dynamics damping="${joints_damping}"/>
     <limit effort="51" velocity="${225/180*pi}" lower="${-2*pi}" upper="${2*pi}"/>
-    <!-- <limit effort="51" velocity="${225/180*pi}" lower="${-177.6 * pi_per_deg}" upper="${177.6 * pi_per_deg}"/> -->
   </joint>
   </xacro:macro>
