Commit message: rework files for mock dual arm launch

File: kassow_kord_bringup/srdf/kassow_kord.srdf.xacro (robot description, xacro)
@@ -1,31 +1,6 @@
 <?xml version="1.0" encoding="UTF-8"?>
-<!--This does not replace URDF, and is not an extension of URDF.
-This is a format for representing semantic information about the robot structure.
-A URDF file must exist for this robot as well, where the joints and the links that are referenced are defined
--->
 <robot name="kassow_kord" xmlns:xacro="http://wiki.ros.org/xacro">
-    <xacro:arg name="robot_name" default="kassow_kord"/>
     <xacro:arg name="prefix" default=""/>
-    <!--GROUPS- Representation of a set of joints and links. This can be useful for specifying DOF to plan for, defining arms, end effectors, etc-->
-    <!--LINKS- When a link is specified, the parent joint of that link (if it exists) is automatically included-->
-    <!--JOINTS- When a joint is specified, the child link of that joint (which will always exist) is automatically included-->
-    <!--CHAINS- When a chain is specified, all the links along the chain (including endpoints) are included in the group. Additionally, all the joints that are parents to included links are also included. This means that joints along the chain and the parent joint of the base link are included in the group-->
-    <!--SUBGROUPS- Groups can also be formed by referencing to already defined group names-->
-    <group name="manipulator">
-        <chain base_link="base" tip_link="end_effector"/>
-    </group>
-    <!--DISABLE COLLISIONS- By default it is assumed that any link of the robot could potentially come into collision with any other link in the robot. This tag disables collision checking between a specified pair of links. -->
-    <!-- Robot -->
-    <disable_collisions link1="base" link2="link1" reason="Adjacent" />
-    <disable_collisions link1="link1" link2="linkJ2" reason="Adjacent" />
-    <disable_collisions link1="link1" link2="link2" reason="Adjacent" />
-    <disable_collisions link1="linkJ2" link2="link2" reason="Adjacent" />
-    <disable_collisions link1="link2" link2="link3" reason="Adjacent" />
-    <disable_collisions link1="link3" link2="linkJ4" reason="Adjacent" />
-    <disable_collisions link1="linkJ4" link2="link4" reason="Adjacent" />
-    <disable_collisions link1="link4" link2="link5" reason="Adjacent" />
-    <disable_collisions link1="link5" link2="linkJ6" reason="Adjacent" />
-    <disable_collisions link1="link5" link2="link6" reason="Adjacent" />
-    <disable_collisions link1="linkJ6" link2="link6" reason="Adjacent" />
-    <disable_collisions link1="link6" link2="end_effector" reason="Adjacent" />
+    <xacro:include filename="$(find kassow_kord_bringup)/srdf/kassow_kord_macro.srdf.xacro"/>
+    <xacro:kassow_kord_srdf prefix="$(arg prefix)"/>
 </robot>

File: kassow_kord_bringup/urdf/kassow_kord.ros2_control.xacro (robot description, xacro)
@@ -26,5 +26,5 @@
         </xacro:unless>
       </hardware>
-      <joint name="joint_1">
+      <joint name="${prefix}_joint_1">
         <command_interface name="position"/>
         <command_interface name="velocity"/>
@@ -35,5 +35,5 @@
         <state_interface name="effort"/>
       </joint>
-      <joint name="joint_2">
+      <joint name="${prefix}_joint_2">
         <command_interface name="position"/>
         <command_interface name="velocity"/>
@@ -44,5 +44,5 @@
         <state_interface name="effort"/>
       </joint>
-      <joint name="joint_3">
+      <joint name="${prefix}_joint_3">
         <command_interface name="position"/>
         <command_interface name="velocity"/>
@@ -53,5 +53,5 @@
         <state_interface name="effort"/>
       </joint>
-      <joint name="joint_4">
+      <joint name="${prefix}_joint_4">
         <command_interface name="position"/>
         <command_interface name="velocity"/>
@@ -62,5 +62,5 @@
         <state_interface name="effort"/>
       </joint>
-      <joint name="joint_5">
+      <joint name="${prefix}_joint_5">
         <command_interface name="position"/>
         <command_interface name="velocity"/>
@@ -71,5 +71,5 @@
         <state_interface name="effort"/>
       </joint>
-      <joint name="joint_6">
+      <joint name="${prefix}_joint_6">
         <command_interface name="position"/>
         <command_interface name="velocity"/>
@@ -80,5 +80,5 @@
         <state_interface name="effort"/>
       </joint>
-      <joint name="joint_7">
+      <joint name="${prefix}_joint_7">
         <command_interface name="position"/>
         <command_interface name="velocity"/>

File: kassow_kord_bringup/urdf/kassow_kord.urdf.xacro (robot description, xacro)
@@ -1,5 +1,5 @@
 <?xml version="1.0"?>
 <robot xmlns:xacro="http://www.ros.org/wiki/xacro" name="kassow_kord">
-  <xacro:arg name="prefix" default=""/>
+  <xacro:arg name="prefix" default="kassow"/>
   <xacro:arg name="use_mock_hardware" default="true"/>
   <xacro:arg name="ip_address" default="10.28.28.11"/>
@@ -7,11 +7,13 @@
   <xacro:arg name="session_id" default="1"/>
   <xacro:include filename="$(find kassow_kord_bringup)/urdf/common/inertials.xacro" />
+  <xacro:include filename="$(find kassow_kord_bringup)/urdf/common/materials.xacro" />
   <xacro:include filename="$(find kassow_kord_description)/kr810/urdf/kr810_description.urdf.xacro"/>
   <xacro:include filename="$(find kassow_kord_bringup)/urdf/kassow_kord.ros2_control.xacro"/>
-  <!-- Add robot URDF -->
-  <xacro:kr810_description/>
-  <!-- Add ros2_control hardware -->
+  <link name="world"/>
+  <xacro:kr810_description prefix="$(arg prefix)" parent="world">
+    <origin xyz="0 0 0" rpy="0 0 0"/>
+  </xacro:kr810_description>
   <xacro:kassow_kord_ros2_control
-    name="kassow_kord_control"
+    name="$(arg prefix)"
     prefix="$(arg prefix)"
     use_mock_hardware="$(arg use_mock_hardware)"

File: kassow_kord_description/kr810/urdf/kr810_description.urdf.xacro (robot description, xacro)
@@ -1,21 +1,5 @@
 <?xml version="1.0" ?>
 <robot name="kr2_robot_a810" model="a810" model-revision="051020-0" mechanical-revision="5" features="TIO" xmlns:xacro="http://www.ros.org/wiki/xacro">
-  <xacro:macro name="kr810_description">
-  <!-- materials -->
-  <material name="gray">
-    <color rgba="0.5 0.5 0.5 1.0"/>
-  </material>
-  <material name="dark_gray">
-    <color rgba="0.3 0.3 0.3 1.0"/>
-  </material>
-  <material name="light_gray">
-    <color rgba="0.7 0.7 0.7 1.0"/>
-  </material>
-  <material name="black">
-    <color rgba="0.1 0.1 0.1 1.0"/>
-  </material>
-  <material name="orange">
-    <color rgba="${255/255} ${108/255} ${10/255} 1.0"/>
-  </material>
+  <xacro:macro name="kr810_description" params="prefix parent *origin">
   <!-- globals -->
   <xacro:property name="joints_damping" value="0.1" />
@@ -66,6 +50,5 @@
     </collision>
   </xacro:macro>
-  <link name="world"/>
-  <link name="base">
+  <link name="${prefix}_base">
     <xacro:property name="base_outer_radius" value="${ 80 * scale}" />
     <xacro:property name="base_inner_radius" value="${ 60 * scale}" />
@@ -87,5 +70,5 @@
       scale="0.001 0.001 0.001"/>
   </link>
-  <link name="link1">
+  <link name="${prefix}_link1">
     <xacro:property name="link1_radius" value="${ 60 * scale}" />
     <xacro:property name="link1_length" value="${ 308.7 * scale - 35 * scale}" />
@@ -107,5 +90,5 @@
       scale="0.001 0.001 0.001"/>
   </link>
-  <link name="linkJ2">
+  <link name="${prefix}_linkJ2">
     <xacro:property name="cylinderJ2_radius"   value="${15 * scale}"   />
     <xacro:property name="cylinderJ2_height"   value="${120 * scale}"   />
@@ -124,5 +107,5 @@
     </inertial>
   </link>
-  <link name="link2">
+  <link name="${prefix}_link2">
     <xacro:property name="link2_radius"   value="${ 45.0 * scale}"   />
     <xacro:property name="link2_length"   value="${ 274.0 * scale}"   />
@@ -142,5 +125,5 @@
       scale="0.001 0.001 0.001"/>
   </link>
-  <link name="link3">
+  <link name="${prefix}_link3">
     <xacro:property name="link3_radius"        value="${  45.0 * scale}" />
     <xacro:property name="link3_length"        value="${ 142.9 * scale}" />
@@ -163,5 +146,5 @@
       scale="0.001 0.001 0.001"/>
   </link>
-  <link name="linkJ4">
+  <link name="${prefix}_linkJ4">
     <xacro:property name="cylinderJ4_radius"   value="${15.0 * scale}"   />
     <xacro:property name="cylinderJ4_height"   value="${100 * scale}"   />
@@ -180,5 +163,5 @@
     </inertial>
   </link>
-  <link name="link4">
+  <link name="${prefix}_link4">
     <xacro:property name="link4_radius"   value="${  40.0 * scale}" />
     <xacro:property name="link4_length"   value="${ 271.0 * scale}" />
@@ -198,5 +181,5 @@
       scale="0.001 0.001 0.001"/>
   </link>
-  <link name="link5">
+  <link name="${prefix}_link5">
     <xacro:property name="link5_radius"   value="${  40.0 * scale}" />
     <xacro:property name="link5_length"   value="${ 103.5 * scale}" />
@@ -216,5 +199,5 @@
       scale="0.001 0.001 0.001"/>
   </link>
-  <link name="linkJ6">
+  <link name="${prefix}_linkJ6">
     <xacro:property name="cylinderJ6_radius"   value="${ 15.0 * scale}"   />
     <xacro:property name="cylinderJ6_height"   value="${ 110.0 * scale}"  />
@@ -233,5 +216,5 @@
     </inertial>
   </link>
-  <link name="link6">
+  <link name="${prefix}_link6">
     <xacro:property name="link6_radius"   value="${ 35.0 * scale}" />
     <xacro:property name="link6_length"   value="${ 66.5 * scale}" />
@@ -251,5 +234,5 @@
       scale="0.001 0.001 0.001"/>
   </link>
-  <link name="end_effector">
+  <link name="${prefix}_end_effector">
     <xacro:property name="end_effector_outer_radius" value="${ 35.5 * scale}" />
     <xacro:property name="end_effector_outer_length" value="${ 5.0 * scale}" />
@@ -272,11 +255,12 @@
   </link>
   <!-- joints -->
-  <joint name="dummy" type="fixed">
-    <parent link="world"/>
-    <child link="base"/>
-  </joint>
-  <joint name="joint_1" type="revolute">
-    <parent link="base"/>
-    <child link="link1"/>
+  <joint name="${prefix}_parent_link" type="fixed">
+    <xacro:insert_block name="origin" />
+    <parent link="${parent}"/>
+    <child link="${prefix}_base"/>
+  </joint>
+  <joint name="${prefix}_joint_1" type="revolute">
+    <parent link="${prefix}_base"/>
+    <child link="${prefix}_link1"/>
     <origin rpy="0 0 0" xyz="0 0 ${base_inner_height + base_outer_height}"/>
     <axis xyz="0 0 1"/>
@@ -287,7 +271,7 @@
   <xacro:property name="joint1_yoffset"  value="${   0.0 * scale}" />
   <xacro:property name="joint1_zoffset"  value="${ 308.7 * scale - 35 * scale}" />
-  <joint name="joint_2" type="revolute">
-    <parent link="link1"/>
-    <child link="linkJ2"/>
+  <joint name="${prefix}_joint_2" type="revolute">
+    <parent link="${prefix}_link1"/>
+    <child link="${prefix}_linkJ2"/>
     <origin rpy="0 0 0" xyz="${joint1_xoffset} ${joint1_yoffset} ${joint1_zoffset}"/>
     <axis xyz="0 1 0"/>
@@ -297,12 +281,12 @@
   <xacro:property name="jointPL2_xoffset"  value="${  -50.0 * scale}" />
   <xacro:property name="jointPL2_yoffset"  value="${  -85.7 * scale}" />
-  <joint name="jointPL2" type="fixed">
-    <parent link="linkJ2"/>
-    <child link="link2"/>
+  <joint name="${prefix}_jointPL2" type="fixed">
+    <parent link="${prefix}_linkJ2"/>
+    <child link="${prefix}_link2"/>
     <origin rpy="0 0 0" xyz="${jointPL2_xoffset} ${jointPL2_yoffset} 0"/>
   </joint>
-  <joint name="joint_3" type="revolute">
-    <parent link="link2"/>
-    <child link="link3"/>
+  <joint name="${prefix}_joint_3" type="revolute">
+    <parent link="${prefix}_link2"/>
+    <child link="${prefix}_link3"/>
     <origin rpy="0 0 0" xyz="0 0 ${link2_length}"/>
     <axis xyz="0 0 1"/>
@@ -313,7 +297,7 @@
   <xacro:property name="joint3_yoffset"  value="${ 0.0 * scale}" />
   <xacro:property name="joint3_zoffset"  value="${ 142.9 * scale}" />
-  <joint name="joint_4" type="revolute">
-    <parent link="link3"/>
-    <child link="linkJ4"/>
+  <joint name="${prefix}_joint_4" type="revolute">
+    <parent link="${prefix}_link3"/>
+    <child link="${prefix}_linkJ4"/>
     <origin rpy="0 0 0" xyz="${joint3_xoffset} ${joint3_yoffset} ${joint3_zoffset}"/>
     <axis xyz="0 1 0"/>
@@ -324,12 +308,12 @@
   <xacro:property name="jointPL4_yoffset"  value="${ 84.05 * scale}" />
   <xacro:property name="jointPL4_zoffset"  value="${ 0.0 * scale}" />
-  <joint name="jointPL4" type="fixed">
-    <parent link="linkJ4"/>
-    <child link="link4"/>
+  <joint name="${prefix}_jointPL4" type="fixed">
+    <parent link="${prefix}_linkJ4"/>
+    <child link="${prefix}_link4"/>
     <origin rpy="0 0 0" xyz="${jointPL4_xoffset} ${jointPL4_yoffset} ${jointPL4_zoffset}"/>
   </joint>
-  <joint name="joint_5" type="revolute">
-    <parent link="link4"/>
-    <child link="link5"/>
+  <joint name="${prefix}_joint_5" type="revolute">
+    <parent link="${prefix}_link4"/>
+    <child link="${prefix}_link5"/>
     <origin rpy="0 0 0" xyz="0 0 ${link4_length}"/>
     <axis xyz="0 0 1"/>
@@ -338,7 +322,7 @@
   </joint>
   <xacro:property name="joint5_zoffset"  value="${ 103.5 * scale}" />
-  <joint name="joint_6" type="revolute">
-    <parent link="link5"/>
-    <child link="linkJ6"/>
+  <joint name="${prefix}_joint_6" type="revolute">
+    <parent link="${prefix}_link5"/>
+    <child link="${prefix}_linkJ6"/>
     <origin rpy="0 0 0" xyz="0 0 ${joint5_zoffset}"/>
     <axis xyz="0 1 0"/>
@@ -347,13 +331,13 @@
   </joint>
   <xacro:property name="jointPL6_yoffset"  value="${ 111.0 * scale}" />
-  <joint name="jointPL6" type="fixed">
-    <parent link="linkJ6"/>
-    <child link="link6"/>
+  <joint name="${prefix}_jointPL6" type="fixed">
+    <parent link="${prefix}_linkJ6"/>
+    <child link="${prefix}_link6"/>
     <origin rpy="0 0 0" xyz="0 ${jointPL6_yoffset} 0"/>
   </joint>
   <xacro:property name="joint6_zoffset"  value="${ 108.0 * scale}" />
-  <joint name="joint_7" type="revolute">
-    <parent link="link6"/>
-    <child link="end_effector"/>
+  <joint name="${prefix}_joint_7" type="revolute">
+    <parent link="${prefix}_link6"/>
+    <child link="${prefix}_end_effector"/>
     <origin rpy="0 0 0" xyz="0 0 ${joint6_zoffset}"/>
     <axis xyz="0 0 1"/>
